File: PCB/Kicad/Main-PCB/ESP32_MIDI_v3a/ESP32_MIDI_v3a.kicad_pcb (KiCad board)
At the start: 2 copper layers, 171 x 28 mm, 28 parts

Commit message: firmware
Parts:
- removed H3, H4: MountingHole, MountingHole:MountingHole_3.2mm_M3_ISO14580
- removed RV4: R_Potentiometer_Dual, ih_kicad:potentiometer_wheel_10mm_SMD-shield
- added U1: LSM6DS3_Breakout, ih_kicad:LSM6DS3_Breakout_oneSide, F.Cu at (176.0, 98.5)
Connections:
- D1 pad 4: /SCL -> /D1
Routing:
- net /SCL: track 172.8 -> 50.3 mm, vias 1 -> 2
- net /D1: track 57.3 -> 171.7 mm, vias 0 -> 2
- net /SDA: track 0.00 -> 35.2 mm
- net GND: track 820.4 -> 815.1 mm
- net +3.3V: track 203.0 -> 198.9 mm, vias 2 -> 3
- net /A4: track 72.9 -> 70.7 mm
- net /A5: track 142.5 -> 140.4 mm
- net /D0: track 114.5 -> 115.9 mm
- net /A10: track 161.0 -> 162.2 mm
