File: PCB/Kicad/Main-PCB/ESP32_MIDI_v3a/ESP32_MIDI_v3a.kicad_sch (KiCad schematic)
At the start: 26 parts

Commit message: Jan 10 commit - up to v4
Parts:
- removed D1: WS2812B, LED_THT:LED_D5.0mm-4_RGB_Wide_Pins, symbol LED:WS2812B
- removed H17: MountingHole, MountingHole:MountingHole_3.2mm_M3, symbol Mechanical:MountingHole
- removed RV3: R_Potentiometer_Dual, ih_kicad:potentiometer_wheel_16mm, symbol Device:R_Potentiometer_Dual
- added D1, D2: WS2812B, LED_THT:LED_D5.0mm-4_RGB_Wide_Pins, symbol hattwick:WS2812B_THT_5MM
- added RV2, RV4: R_Potentiometer_Dual, ih_kicad:potentiometer_wheel_10mm_SMD-shield, symbol hattwick:R_Potentiometer_Dual_Wheel
- added TP12: TestPoint, ih_kicad:recorder-touchpad-alt-up, symbol Connector:TestPoint
- H1, H13, H14, H15, H16, H18, H2: footprint MountingHole:MountingHole_3.2mm_M3 -> MountingHole:MountingHole_4.5mm
- H3, H4, H5, H6: footprint MountingHole:MountingHole_3.2mm_M3 -> MountingHole:MountingHole_3.2mm_M3_ISO14580
- TP8: footprint ih_kicad:recorder-touchtrack -> ih_kicad:recorder-touchpad-alt-up
- TP9: footprint ih_kicad:recorder-touchtrack -> ih_kicad:recorder-touchtrack_120mm
Connections:
- net +3.3V: now also D1.3 (VDD), D2.3 (VDD), RV2.1 (1A), RV4.1 (1A)
- net A5: now also TP8.1, RV4.6 (Shield); no longer TP9.1
- net A6: now also TP9.1; no longer TP8.1
- net D0: now also RV2.4 (1-Wiper)
- net D1: now also RV4.4 (1-Wiper)
- net GND: now also D1.2 (VSS), D2.2 (VSS), RV2.5 (Common), RV4.5 (Common)
- net SCL: now also D1.4 (DIN)
- net D2 renamed A10
- net A10: now also RV2.6 (Shield), TP12.1
- new net: D1.1 (DOUT), D2.4 (DIN)
Other:
- moved on the sheet: TP10, TP2, TP3, TP4, TP5, TP6, TP7, TP8, TP9
