File: PCB/Kicad/Main-PCB/ESP32_MIDI_v3a/ESP32_MIDI_v3a.kicad_sch (KiCad schematic)
At the start: 28 parts

Commit message: firmware
Parts:
- removed H3, H4: MountingHole, MountingHole:MountingHole_3.2mm_M3_ISO14580, symbol Mechanical:MountingHole
- removed RV4: R_Potentiometer_Dual, ih_kicad:potentiometer_wheel_10mm_SMD-shield, symbol hattwick:R_Potentiometer_Dual_Wheel
- added U1: LSM6DS3_Breakout, ih_kicad:LSM6DS3_Breakout_oneSide, symbol LSM6DS3_Breakout:LSM6DS3_Breakout
Connections:
- net +3.3V: now also U1.1 (VIN)
- net D1: now also D1.4 (DIN)
- net GND: now also U1.3 (GND)
- net SCL: now also U1.4 (SCL); no longer D1.4 (DIN)
- net SDA: now also U1.5 (SDA)
