File: PCB/Kicad/ESP32_laptop-strip.kicad_pcb/ESP32_laptop-strip.kicad_pcb.kicad_pcb (KiCad board)
At the start: 2 copper layers, 250 x 100.5 mm, 29 parts, among them SW10 RotaryEncoder, SW9 RotaryEncoder

Commit message: update all kicad designs for week 1
Parts:
- removed C7, C8, C9: 0.1uF, Capacitor_SMD:C_0805_2012Metric_Pad1.18x1.45mm_HandSolder
- removed D1, D2, D3, D4: WS2812B, LED_SMD:LED_WS2812B_PLCC4_5.0x5.0mm_P3.2mm
- added C6: 10nF, Capacitor_SMD:C_0805_2012Metric_Pad1.18x1.45mm_HandSolder, F.Cu at (50.5, 101.5)
- added H15: MountingHole_Pad, MountingHole:MountingHole_4.3mm_M4_DIN965_Pad, F.Cu at (182.5, 118.0)
- added J1: Conn_01x03_Pin, ih_kicad:WS2812_PADS, F.Cu at (78.2, 105.0)
- added R1: R_Small, Resistor_SMD:R_0805_2012Metric_Pad1.20x1.40mm_HandSolder, F.Cu at (59.5, 101.5)
- added U1: 74AHCT1G125, Package_TO_SOT_SMD:TSOT-23-5_HandSoldering, F.Cu at (45.5, 103.0)
- H10, H11, H12, H13, H14, H7, H8, H9: footprint MountingHole:MountingHole_4.3mm_M4 -> MountingHole:MountingHole_4.3mm_M4_DIN965_Pad
- SW10, SW9: footprint Rotary_Encoder:RotaryEncoder_Bourns_Vertical_PEL12D-4xxxF-Sxxxx -> ih_kicad:RotaryEncoder_Vertical_10mm
- moved H2 182.0 mm to (45.5, 120.5)
- moved C2 163.1 mm to (23.5, 123.5), turned to 0 degrees
- moved C1 138.7 mm to (66.0, 110.0), turned to -90 degrees
- moved C3 138.4 mm to (66.0, 114.0), turned to -90 degrees
- moved H1 124.1 mm to (150.5, 104.0)
- moved H6 107.4 mm to (238.5, 102.0)
- moved H5 78.8 mm to (155.0, 119.0)
- moved C4 74.4 mm to (225.5, 114.0), turned to 90 degrees
- moved C5 73.3 mm to (225.5, 110.0), turned to 90 degrees
- moved H10 71.7 mm to (92.5, 118.0)
- moved H4 65.5 mm to (239.0, 121.0)
- moved H13 57.3 mm to (200.5, 118.0)
- moved H14 56.0 mm to (128.5, 118.0)
- moved H9 48.5 mm to (74.5, 118.0)
- moved H12 44.2 mm to (218.5, 119.0)
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Connections:
- U2 pad 10: /EncA2 -> /DI
- U2 pad 11: /EncB2 -> /EncA2
- U2 pad 12: /A8 -> /EncB2
- U2 pad 14: /D0 -> /T0
- U2 pad 15: unconnected-(U2-GPIO12/ADC2_CH1-Pad15) -> /T2
- U2 pad 16: unconnected-(U2-GPIO13/ADC2_CH2-Pad16) -> /A8
- U2 pad 17: /DI -> /EncB1
- U2 pad 18: unconnected-(U2-GPIO43/U0TXD-Pad18) -> /EncA1
- U2 pad 8: /EncA1 -> /T1
- U2 pad 9: /EncB1 -> /T4
Routing:
- net GND: track 0.00 -> 317.3 mm, vias 0 -> 12
- net /EncA2: track 0.00 -> 214.9 mm
- net /EncB2: track 0.00 -> 207.0 mm
- net /A9: track 0.00 -> 200.2 mm
- net /T0: track 0.00 -> 183.4 mm
- net /T2: track 0.00 -> 168.1 mm
- net /A8: track 0.00 -> 150.7 mm
- net /A0: track 0.00 -> 132.6 mm
- net /T1: track 0.00 -> 99.8 mm
- net /A1: track 0.00 -> 93.1 mm
- net +5V: track 0.00 -> 87.7 mm, vias 0 -> 3
- net /A3: track 0.00 -> 67.3 mm
- net /EncA1: track 0.00 -> 53.4 mm
- net /A2: track 0.00 -> 51.1 mm
- net /EncB1: track 0.00 -> 48.4 mm
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Other:
- board size 250 x 100.5 mm -> 224.5 x 100 mm
- board text added: "ESP32_laptop-strip v1"
- board text removed: "ESP32_laptop-midi v1"
