File: PCB/Kicad/ESP32_laptop-strip.kicad_pcb/ESP32_laptop-strip.kicad_pcb.kicad_sch (KiCad schematic)
At the start: 29 parts, among them SW10 RotaryEncoder, SW9 RotaryEncoder

Commit message: update all kicad designs for week 1
Parts:
- removed C7, C8, C9: 0.1uF, Capacitor_SMD:C_0805_2012Metric_Pad1.18x1.45mm_HandSolder, symbol Device:C
- removed D1, D2, D3, D4: WS2812B, LED_SMD:LED_WS2812B_PLCC4_5.0x5.0mm_P3.2mm, symbol LED:WS2812B
- added C6: 10nF, Capacitor_SMD:C_0805_2012Metric_Pad1.18x1.45mm_HandSolder, symbol Device:C
- added H15: MountingHole_Pad, MountingHole:MountingHole_4.3mm_M4_DIN965_Pad, symbol Mechanical:MountingHole_Pad
- added J1: Conn_01x03_Pin, ih_kicad:WS2812_PADS, symbol Connector:Conn_01x03_Pin
- added R1: R_Small, Resistor_SMD:R_0805_2012Metric_Pad1.20x1.40mm_HandSolder, symbol Device:R_Small
- added U1: 74AHCT1G125, Package_TO_SOT_SMD:TSOT-23-5_HandSoldering, symbol 74xGxx:74AHCT1G125
- H10, H11, H12, H13, H14, H7, H8, H9: footprint MountingHole:MountingHole_4.3mm_M4 -> MountingHole:MountingHole_4.3mm_M4_DIN965_Pad
- SW10, SW9: footprint Rotary_Encoder:RotaryEncoder_Bourns_Vertical_PEL12D-4xxxF-Sxxxx -> ih_kicad:RotaryEncoder_Vertical_10mm
Connections:
- net +5V: now also C6.1, J1.3 (Pin_3), U1.5 (VCC)
- net A0: no longer H10.1, H11.1, H12.1, H13.1, H14.1, H8.1, H9.1
- net A1: now also H8.1
- net A2: now also H9.1
- net A3: now also H10.1
- net A8: now also H11.1, U2.16 (GPIO13/ADC2_CH2); no longer U2.12 (GPIO9/ADC1_CH8)
- net A9: now also H12.1
- net DI: now also U2.10 (GPIO7/ADC1_CH6), U1.2; no longer U2.17 (GPIO44/U0RXD)
- net EncA1: now also U2.18 (GPIO43/U0TXD); no longer U2.8 (GPIO5/ADC1_CH4)
- net EncA2: now also U2.11 (GPIO8/ADC1_CH7); no longer U2.10 (GPIO7/ADC1_CH6)
- net EncB1: now also U2.17 (GPIO44/U0RXD); no longer U2.9 (GPIO6/ADC1_CH5)
- net EncB2: now also U2.12 (GPIO9/ADC1_CH8); no longer U2.11 (GPIO8/ADC1_CH7)
- net GND: now also C6.2, J1.1 (Pin_1), U1.1, U1.3 (GND)
- net T2: now reaches U2.15 (GPIO12/ADC2_CH1)
- net T2: now also H15.1
- net D0 renamed T0
- net T0: now also H13.1
- new net: J1.2 (Pin_2), R1.2
- new net: R1.1, U1.4
- new net T1: H14.1, U2.8 (GPIO5/ADC1_CH4)
- new net T4: U2.9 (GPIO6/ADC1_CH5)
Other:
- moved on the sheet: H10, H11, H12, H13, H14, H7, H8, H9
