File: PCB/Kicad/Main-PCB/ESP32_MIDI_Summer25_FRETS_v2/ESP32_MIDI_Summer25_FRETS_v2.kicad_pcb (KiCad board)
At the start: 2 copper layers, 28 parts, among them J1 Conn_01x01_Pin, J3 IDC_5x2, U1 MPR121_Breakout

Commit message: update all kicad designs for week 1
Parts:
- removed H20, H21, H22, H23, H24, H25, H26, H27, H28, H29: MountingHole_Pad, MountingHole:MountingHole_6.4mm_M6_DIN965_Pad_TopBottom
- removed J3: IDC_5x2, Connector_IDC:IDC-Header_2x05_P2.54mm_Vertical
- added H3: MountingHole_Pad, MountingHole:MountingHole_6.4mm_M6_DIN965_Pad_TopBottom, F.Cu at (54.0, 48.5)
- J1: value Conn_01x01_Pin -> Conn_01x04_Pin; footprint ih_kicad:recorder-touchtrack_120mm -> Connector_PinHeader_2.54mm:PinHeader_1x04_P2.54mm_Horizontal
- moved J1 141.3 mm to (281.0, 45.5)
- moved H19 83.2 mm to (274.0, 49.0)
- moved H18 78.1 mm to (254.0, 48.5)
- moved H17 73.0 mm to (234.0, 48.5)
- moved H16 68.0 mm to (214.0, 48.5)
- moved H15 63.1 mm to (194.0, 48.5)
- moved H14 58.5 mm to (174.0, 48.5)
- moved U1 58.2 mm to (257.0, 50.0), turned to 180 degrees
- moved H13 54.1 mm to (154.0, 48.5)
- moved H9 53.8 mm to (283.7, 40.1)
- moved H12 50.1 mm to (134.0, 48.5)
- moved H10 47.9 mm to (278.7, 74.6)
- moved H11 46.5 mm to (114.0, 48.5)
- moved H7 42.5 mm to (94.0, 49.5)
- moved H8 41.0 mm to (74.0, 48.5)
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Connections:
- H11 pad 1: /p3 -> /p11
- H12 pad 1: /p4 -> /p7
- H13 pad 1: /p5 -> /p1
- H14 pad 1: /p6 -> /p2
- H15 pad 1: /p7 -> /p3
- H16 pad 1: /p8 -> /p4
- H17 pad 1: /p9 -> /p5
- H18 pad 1: /p10 -> /p6
- H19 pad 1: /p11 -> /p0
- H7 pad 1: /p2 -> /p10
- H8 pad 1: /p1 -> /p9
- J1 pad 1: /p12 -> GND
- U1 pad 16: /p11 -> /p9
- U1 pad 18: /p9 -> /p11
- U1 pad 6: (no net) -> unconnected-(U1-GND-Pad6)
- U1 pad 7: unconnected-(U1-p1-Pad7) -> /p0
Routing:
- net /p6: track 164.9 -> 3.90 mm
- net /p1: track 285.0 -> 128.0 mm
- net /p2: track 246.9 -> 105.8 mm
- net /p3: track 216.5 -> 81.7 mm
- net /p4: track 186.0 -> 61.1 mm
- net /p5: track 160.9 -> 40.7 mm
- net /p11: track 24.6 -> 127.3 mm
- net /p8: track 140.6 -> 199.8 mm
- net /p9: track 124.0 -> 174.9 mm
- net /p7: track 153.7 -> 117.2 mm
- net /SCL: track 11.2 -> 34.0 mm
- net GND: track 38.1 -> 59.2 mm
- net +3.3V: track 30.5 -> 43.1 mm
- net /p12: track 7.74 -> 0.00 mm
- net /p0: track 0.00 -> 6.52 mm
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Other:
- board outline added: 237.5 x 25 mm
- board text added: "3v"
- board text added: "CL"
- board text added: "Creativitas Frets v2"
- board text added: "DA"
- board text added: "G"
- board text removed: "3v3"
- board text removed: "Creativitas Frets v1"
- board text removed: "IRQ"
- board text removed: "SCL"
- board text removed: "SDA"
