File: PCB/Kicad/Main-PCB/ESP32_MIDI_Summer25_FRETS_v2/ESP32_MIDI_Summer25_FRETS_v2.kicad_sch (KiCad schematic)
At the start: 28 parts, among them J1 Conn_01x01_Pin, J3 IDC_5x2, U1 MPR121_Breakout

Commit message: update all kicad designs for week 1
Parts:
- removed H20, H21, H22, H23, H24, H25, H26, H27, H28, H29: MountingHole_Pad, MountingHole:MountingHole_6.4mm_M6_DIN965_Pad_TopBottom, symbol Mechanical:MountingHole_Pad
- removed J1: Conn_01x01_Pin, ih_kicad:recorder-touchtrack_120mm, symbol Connector:Conn_01x01_Pin
- removed J3: IDC_5x2, Connector_IDC:IDC-Header_2x05_P2.54mm_Vertical, symbol Connector_Generic:Conn_02x05_Odd_Even
- added H3: MountingHole_Pad, MountingHole:MountingHole_6.4mm_M6_DIN965_Pad_TopBottom, symbol Mechanical:MountingHole_Pad
- added J1: Conn_01x04_Pin, Connector_PinHeader_2.54mm:PinHeader_1x04_P2.54mm_Horizontal, symbol Connector:Conn_01x04_Pin
Connections:
- net +3.3V: now also J1.2 (Pin_2)
- net GND: now also J1.1 (Pin_1)
- net SCL: now also J1.3 (Pin_3)
- net SDA: now also J1.4 (Pin_4)
- net p1: now also H13.1; no longer H8.1
- net p10: now also H7.1; no longer H18.1
- net p11: now also H11.1, U1.18 (T11); no longer H19.1, U1.16 (p10)
- net p2: now also H14.1; no longer H7.1
- net p3: now also H15.1; no longer H11.1
- net p4: now also H16.1; no longer H12.1
- net p5: now also H17.1; no longer H13.1
- net p6: now also H18.1; no longer H14.1
- net p7: now also H12.1; no longer H15.1
- net p8: now also H3.1; no longer H16.1
- net p9: now also H8.1, U1.16 (T9); no longer H17.1, U1.18 (p12)
- net p0: now reaches U1.7 (T0)
- net p0: now also H19.1
Other:
- note added: "v2 fixes: + 4 pin jumper cable header - JST XH? - revise capsense placement - check holes for connection to GTR - fix capsense breakout pins - update cap hole with silkscreen"
- note removed: "v2 fixes: - 4 pin jumper cable header - JST XH? - revise capsense placement - check holes for connection to GTR - fix capsense breakout pins - update cap hole with silkscreen"
