File: PCB/Kicad/Main-PCB/Sum25_GTR/Sum25_GTR.kicad_sch (KiCad schematic)
At the start: 20 parts, among them J3 IDC_5x2, U4 DRV5055A2xLPGxQ1, U5 DRV5055A2xLPGxQ1

Commit message: update all kicad designs for week 1
Parts:
- removed J3: IDC_5x2, Connector_IDC:IDC-Header_2x05_P2.54mm_Vertical, symbol Connector_Generic:Conn_02x05_Odd_Even
- added H11, H12, H13, H14, H15, H16: MountingHole, MountingHole:MountingHole_3.2mm_M3, symbol Mechanical:MountingHole
- added J1, J2: Conn_01x04_Pin, Connector_PinSocket_2.54mm:PinSocket_1x04_P2.54mm_Vertical, symbol Connector:Conn_01x04_Pin
- H1, H2, H3, H5: footprint MountingHole:MountingHole_4.3mm_M4 -> MountingHole:MountingHole_3.2mm_M3
Connections:
- net +3.3V: now also J1.2 (Pin_2), J2.2 (Pin_2)
- net A2: no longer RV1.2
- net A3: no longer RV2.2
- net A7: now also RV1.2
- net A9: now also RV2.2; no longer H7.1
- net D0: now also H7.1
- net GND: now also J1.1 (Pin_1), J2.1 (Pin_1)
- net SCL: now also J1.3 (Pin_3), J2.3 (Pin_3)
- net SDA: now also J1.4 (Pin_4), J2.4 (Pin_4)
Other:
- note added: "rev 2.0 fixes - check holes for screws - make sure traces aren't cut by holes + 4-pin JST XH header - check distance between pots and touchposts + m3 screws instead of m4?"
- note removed: "rev 2.0 fixes - check holes for screws - make sure traces aren't cut by holes - 4-pin JST XH header - check distance between pots and touchposts - m3 screws instead of m4?"
