File: PCB/Kicad/Main-PCB/Sum25_Wand_v2/Sum25_Wand_v2.kicad_pcb (KiCad board)
At the start: 2 copper layers, 246 x 30 mm, 22 parts, among them SW1 SW_SPST, SW2 SW_SPST, SW3 SW_SPST, SW4 SW_SPST, U1 74AHCT1G125

Commit message: update all kicad designs for week 1
Parts:
- C1, C2, C3, R1, R2, R3: moved to B.Cu
- RV1, RV2: footprint ih_kicad:potentiometer_wheel_10mm_SMD-shield -> ih_kicad:potentiometer_wheel_10mm
- SW1, SW2, SW3, SW4: footprint Button_Switch_Keyboard:SW_Cherry_MX_1.00u_PCB -> Button_Switch_Keyboard:SW_Cherry_MX_1.00u_Plate
- moved C1 29.8 mm to (195.5, 88.0), turned to -90 degrees
- moved IMU1 29.5 mm to (240.5, 89.6), turned to -90 degrees
- moved U1 17.6 mm to (190.0, 91.5)
- moved R1 14.2 mm to (185.3, 92.0), turned to 180 degrees
- moved SW4 12.1 mm to (188.0, 99.0), turned to 180 degrees
- moved SW3 12.1 mm to (207.1, 99.0), turned to 180 degrees
- moved SW1 12.1 mm to (245.3, 99.0), turned to 180 degrees
- moved C3 6.58 mm to (176.5, 97.0), turned to -90 degrees
- moved R2 5.00 mm to (244.0, 86.0)
- moved R3 3.50 mm to (248.5, 85.9)
- moved RV1 1.00 mm to (182.0, 110.0)
- moved RV2 1.00 mm to (202.0, 110.0)
- moved SW2 0.97 mm to (231.3, 109.2)
Connections:
- RV1 pad 4: /A0 -> /A1
- RV2 pad 4: /A1 -> /A0
- U1 pad 2: /D0 -> /A3
Routing:
- net /D0: track 96.2 -> 0.00 mm
- net /A9: track 172.1 -> 80.6 mm
- net /A3: track 0.00 -> 76.4 mm
- net +3.3V: track 89.3 -> 124.5 mm, vias 0 -> 2
- net /A7: track 44.0 -> 75.1 mm
- net /A1: track 64.2 -> 92.3 mm
- net GND: track 60.3 -> 43.8 mm, vias 8 -> 5
- net /A0: track 88.8 -> 74.6 mm
- net /A6: track 20.6 -> 11.4 mm
- net /A8: track 65.3 -> 58.5 mm
- net +5V: track 291.2 -> 286.0 mm
- net /SDA: track 29.1 -> 33.2 mm
- net Net-(D1-DO): track 18.6 -> 22.5 mm
Other:
- board size 246 x 30 mm -> 245 x 30 mm
- board text added: "0.1uF"
- board text added: "100uF"
- board text added: "2.2k"
- board text added: "220R"
- board text added: "MIDI WAND v2.0"
- board text added: "SCL"
- board text added: "SDA"
- board text removed: "MIDI WAND v1.0"
