File: PCB/Kicad/Main-PCB/Sum25_Wand_v2/Sum25_Wand_v2.kicad_sch (KiCad schematic)
At the start: 22 parts, among them SW1 SW_SPST, SW2 SW_SPST, SW3 SW_SPST, SW4 SW_SPST, U1 74AHCT1G125

Commit message: update all kicad designs for week 1
Parts:
- RV1, RV2: footprint ih_kicad:potentiometer_wheel_10mm_SMD-shield -> ih_kicad:potentiometer_wheel_10mm
- SW1, SW2, SW3, SW4: footprint Button_Switch_Keyboard:SW_Cherry_MX_1.00u_PCB -> Button_Switch_Keyboard:SW_Cherry_MX_1.00u_Plate
Connections:
- net A0: now also RV2.4 (1-Wiper); no longer RV1.4 (1-Wiper)
- net A1: now also RV1.4 (1-Wiper); no longer RV2.4 (1-Wiper)
- net A3: now also U1.2
- net D0: no longer U1.2
Other:
- note added: "V2 fixes + swap order of IMU pins + holes for support pins of potentiometers + tighten holes for mx pins + resistors and capacitors on switch side of PCB"
- note removed: "V2 fixes - swap order of IMU pins - holes for support pins of potentiometers - - tighten holes for mx pins - resistors and capacitors on switch side of PCB"
Changed lines of the file:
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@@
 		)
 	)
-	(text "V2 fixes\n- swap order of IMU pins\n- holes for support pins of potentiometers\n- - tighten holes for mx pins\n- resistors and capacitors on switch side of PCB"
+	(text "V2 fixes\n+ swap order of IMU pins\n+ holes for support pins of potentiometers\n+ tighten holes for mx pins\n+ resistors and capacitors on switch side of PCB"
 		(exclude_from_sim no)
 		(at 22.098 122.682 0)
@@
 		)
 	)
-	(label "A1"
+	(label "A0"
 		(at 171.45 44.45 0)
 		(fields_autoplaced yes)
@@
 		)
 	)
-	(label "D0"
+	(label "A3"
 		(at 24.13 27.94 0)
 		(fields_autoplaced yes)
@@
 		)
 	)
-	(label "A0"
+	(label "A1"
 		(at 171.45 25.4 0)
 		(fields_autoplaced yes)
@@
 			)
 		)
-		(property "Footprint" "Button_Switch_Keyboard:SW_Cherry_MX_1.00u_PCB"
+		(property "Footprint" "Button_Switch_Keyboard:SW_Cherry_MX_1.00u_Plate"
 			(at 231.14 85.09 0)
 			(effects
@@
 			)
 		)
-		(property "Footprint" "Button_Switch_Keyboard:SW_Cherry_MX_1.00u_PCB"
+		(property "Footprint" "Button_Switch_Keyboard:SW_Cherry_MX_1.00u_Plate"
 			(at 231.14 53.34 0)
 			(effects
@@
 			)
 		)
-		(property "Footprint" "Button_Switch_Keyboard:SW_Cherry_MX_1.00u_PCB"
+		(property "Footprint" "Button_Switch_Keyboard:SW_Cherry_MX_1.00u_Plate"
 			(at 231.14 63.5 0)
 			(effects
@@
 			)
 		)
-		(property "Footprint" "ih_kicad:potentiometer_wheel_10mm_SMD-shield"
+		(property "Footprint" "ih_kicad:potentiometer_wheel_10mm"
 			(at 182.88 48.895 0)
 			(effects
@@
 			)
 		)
-		(property "Footprint" "Button_Switch_Keyboard:SW_Cherry_MX_1.00u_PCB"
+		(property "Footprint" "Button_Switch_Keyboard:SW_Cherry_MX_1.00u_Plate"
 			(at 231.14 73.66 0)
 			(effects
@@
 			)
 		)
-		(property "Footprint" "ih_kicad:potentiometer_wheel_10mm_SMD-shield"
+		(property "Footprint" "ih_kicad:potentiometer_wheel_10mm"
 			(at 182.88 29.845 0)
 			(effects
