File: PCB/Kicad/Main-PCB/ESP32_MIDI_Summer25_FRETS_v2_5.kicad_pcb/ESP32_MIDI_Summer25_FRETS_v2_5.kicad_pcb.kicad_pcb (KiCad board)
At the start: 2 copper layers, 209.5 x 25 mm, 18 parts, among them J1 Conn_01x04_Pin, U1 MPR121_Breakout

Commit message: July 26 gerbers
Parts:
- added JP1: Jumper_2_Open, Jumper:SolderJumper-2_P1.3mm_Open_RoundedPad1.0x1.5mm, B.Cu at (251.3, 53.0)
Connections:
- U1 pad 3: GND -> /SCL
- U1 pad 4: /SCL -> /SDA
- U1 pad 5: /SDA -> Net-(JP1-B)
- U1 pad 6: unconnected-(U1-GND-Pad6) -> GND
Routing:
- net /p11: track 123.3 -> 160.9 mm
- net GND: track 59.2 -> 23.1 mm
- net Net-(JP1-B): track 0.00 -> 14.5 mm
- net /p9: track 185.1 -> 176.2 mm
- net +3.3V: track 43.1 -> 48.7 mm
- net /p10: track 147.9 -> 142.4 mm
- net /SCL: track 34.0 -> 36.4 mm
- net /SDA: track 24.9 -> 27.2 mm
- net /p2: track 106.7 -> 104.4 mm
- net /p1: track 129.4 -> 130.7 mm
- net /p0: track 43.8 -> 43.3 mm
Other:
- board text added: "ADD"
- board text added: "Creativitas Frets v2.5b"
- board text added: "Ian Hattwick July '25"
- board text added: "SCL"
- board text added: "SDA"
- board text added: "V+"
- board text removed: "Creativitas Frets v2.5"
- board text removed: "Ian Hattwick Jun '25"
