File: PCB/Kicad/Main-PCB/ESP32_MIDI_Summer25_FRETS_v2_5.kicad_pcb/ESP32_MIDI_Summer25_FRETS_v2_5.kicad_pcb.kicad_sch (KiCad schematic)
At the start: 18 parts, among them J1 Conn_01x04_Pin, U1 MPR121_Breakout

Commit message: July 26 gerbers
Parts:
- added JP1: Jumper_2_Open, Jumper:SolderJumper-2_P1.3mm_Open_RoundedPad1.0x1.5mm, symbol Jumper:Jumper_2_Open
Connections:
- net +3.3V: now also JP1.1 (A)
- net GND: now also U1.6 (GND); no longer U1.3 (SCL)
- net SCL: now also U1.3 (SCL); no longer U1.4 (SDA)
- net SDA: now also U1.4 (SDA); no longer U1.5 (ADD)
- new net: JP1.2 (B), U1.5 (ADD)
Changed lines of the file:
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@@
 	(generator_version "8.0")
 	(paper "A4")
+	(junction
+		(at 176.53 77.47)
+		(diameter 0)
+		(color 0 0 0 0)
+	)
+	(wire
+		(pts
+			(xy 162.56 87.63) (xy 160.02 87.63)
+		)
+		(stroke
+			(width 0)
+			(type default)
+		)
+	)
 	(wire
 		(pts
@@
 	(wire
 		(pts
-			(xy 172.72 82.55) (xy 182.88 82.55)
-		)
-		(stroke
-			(width 0)
-			(type default)
-		)
-	)
-	(wire
-		(pts
 			(xy 201.93 87.63) (xy 207.01 87.63)
 		)
@@
 	(wire
 		(pts
-			(xy 176.53 87.63) (xy 182.88 87.63)
+			(xy 173.99 92.71) (xy 182.88 92.71)
+		)
+		(stroke
+			(width 0)
+			(type default)
+		)
+	)
+	(wire
+		(pts
+			(xy 160.02 87.63) (xy 160.02 77.47)
 		)
 		(stroke
@@
 	(wire
 		(pts
+			(xy 176.53 82.55) (xy 182.88 82.55)
+		)
+		(stroke
+			(width 0)
+			(type default)
+		)
+	)
+	(wire
+		(pts
 			(xy 201.93 77.47) (xy 204.47 77.47)
 		)
@@
 		(pts
 			(xy 201.93 97.79) (xy 207.01 97.79)
+		)
+		(stroke
+			(width 0)
+			(type default)
+		)
+	)
+	(wire
+		(pts
+			(xy 160.02 77.47) (xy 176.53 77.47)
+		)
+		(stroke
+			(width 0)
+			(type default)
+		)
+	)
+	(wire
+		(pts
+			(xy 172.72 87.63) (xy 182.88 87.63)
 		)
 		(stroke
@@
 		)
 	)
-	(label "SDA"
-		(at 177.8 87.63 0)
-		(fields_autoplaced yes)
-		(effects
-			(font
-				(size 1.27 1.27)
-			)
-			(justify left bottom)
-		)
-	)
 	(label "p9"
 		(at 104.14 33.02 0)
@@
 		)
 	)
+	(label "SDA"
+		(at 177.8 85.09 0)
+		(fields_autoplaced yes)
+		(effects
+			(font
+				(size 1.27 1.27)
+			)
+			(justify left bottom)
+		)
+	)
 	(label "p4"
 		(at 204.47 92.71 0)
@@
 	)
 	(label "SCL"
-		(at 177.8 85.09 0)
+		(at 177.8 82.55 0)
 		(fields_autoplaced yes)
 		(effects
@@
 	(symbol
 		(lib_id "power:GND")
-		(at 172.72 82.55 0)
+		(at 173.99 92.71 0)
 		(unit 1)
 		(exclude_from_sim no)
@@
 		(fields_autoplaced yes)
 		(property "Reference" "#PWR02"
-			(at 172.72 88.9 0)
+			(at 173.99 99.06 0)
 			(effects
 				(font
@@
 		)
 		(property "Value" "GND"
-			(at 172.72 87.63 0)
+			(at 173.99 97.79 0)
 			(effects
 				(font
@@
 		)
 		(property "Footprint" ""
-			(at 172.72 82.55 0)
+			(at 173.99 92.71 0)
 			(effects
 				(font
@@
 		)
 		(property "Datasheet" ""
-			(at 172.72 82.55 0)
+			(at 173.99 92.71 0)
 			(effects
 				(font
@@
 		)
 		(property "Description" "Power symbol creates a global label with name \"GND\" , ground"
-			(at 172.72 82.55 0)
+			(at 173.99 92.71 0)
 			(effects
 				(font
@@
 					(unit 1)
 				)
+			)
+		)
+	)
+	(symbol
+		(lib_id "Jumper:Jumper_2_Open")
+		(at 167.64 87.63 0)
+		(unit 1)
+		(exclude_from_sim yes)
+		(in_bom yes)
+		(on_board yes)
+		(dnp no)
+		(fields_autoplaced yes)
+		(property "Reference" "JP1"
+			(at 167.64 81.28 0)
+			(effects
+				(font
+					(size 1.27 1.27)
+				)
+			)
+		)
+		(property "Value" "Jumper_2_Open"
+			(at 167.64 83.82 0)
+			(effects
+				(font
+					(size 1.27 1.27)
+				)
+			)
+		)
+		(property "Footprint" "Jumper:SolderJumper-2_P1.3mm_Open_RoundedPad1.0x1.5mm"
+			(at 167.64 87.63 0)
+			(effects
+				(font
+					(size 1.27 1.27)
+				)
+				(hide yes)
+			)
+		)
+		(property "Datasheet" "~"
+			(at 167.64 87.63 0)
+			(effects
+				(font
+					(size 1.27 1.27)
+				)
+				(hide yes)
+			)
+		)
+		(property "Description" "Jumper, 2-pole, open"
+			(at 167.64 87.63 0)
+			(effects
+				(font
+					(size 1.27 1.27)
+				)
+				(hide yes)
+			)
+		)
+		(pin "1"
+		)
+		(pin "2"
+		)
+		(instances
+			(project ""
+				(path "/41e4c161-2329-4e5f-9dd3-fb5a1db779ba"
+					(reference "JP1")
+					(unit 1)
+				)
